Commit message: feat: fix visual and collision meshes

File: models/ur10.urdf (robot description, URDF)
Before this commit: robot ur10-test, 13 links, 12 joints
Links:
- removed link world
- link base_link_inertia: geometry collision mesh filename=ur10/collision/base.obj; visual mesh filename=ur10/visual/base.gltf
- link forearm_link: geometry collision mesh filename=ur10/collision/forearm.obj; visual mesh filename=ur10/visual/forearm.gltf
- link shoulder_link: geometry collision mesh filename=ur10/collision/shoulder.obj; visual mesh filename=ur10/visual/shoulder.gltf
- link upper_arm_link: geometry collision mesh filename=ur10/collision/upperarm.obj; visual mesh filename=ur10/visual/upperarm.gltf
- link wrist_1_link: geometry collision mesh filename=ur10/collision/wrist1.obj; visual mesh filename=ur10/visual/wrist1.gltf
- link wrist_2_link: geometry collision mesh filename=ur10/collision/wrist2.obj; visual mesh filename=ur10/visual/wrist2.gltf
- link wrist_3_link: geometry collision mesh filename=ur10/collision/wrist3.obj; visual mesh filename=ur10/visual/wrist3.gltf
Joints:
- removed joint base_joint
